File: P4/PCB/MicroMod_tinycar/MicroMod_tinycar.kicad_pcb (KiCad board)
At the start: 2 copper layers, 52.1 x 29.2 mm, 30 parts, among them J1 USB_B_Micro, J2 Conn_01x02, J3 Conn_02x15_Counter_Clockwise, J4 MICROMOD-2222, J5 Conn_02x15_Counter_Clockwise, J6 Conn_02x15_Counter_Clockwise, Q1 DMG2305UX-MicroMod_tinycar_sy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, SW1 SW_SPDT, SW2 SW_Push, U1 MCP73830LT-0AAI_MYY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

Commit message: done with P4
Parts:
- added U7: caster, MicroMod_tinycar_footprint_library:tiny_caster, F.Cu at (160.0, 109.2)
- added U8: MouseBite, MicroMod_tinycar_footprint_library:mouse-bite-2.54mm-slot, F.Cu at (147.3, 118.7)
- U3, U6: moved to B.Cu
- moved U6 2.54 mm to (167.9, 127.9)
- moved U3 2.44 mm to (152.1, 127.9)
- moved C4 0.59 mm to (133.3, 119.0)
- moved Q1 0.40 mm to (139.7, 123.1)
- moved J2 0.38 mm to (139.7, 119.3)
Connections:
- J5 pad 21: Net-(J5-Pad21) -> PWM1
- J6 pad 12: B0- -> B0+
- J6 pad 13: B0+ -> B0-
- J6 pad 14: A0+ -> A0-
- J6 pad 15: A0- -> A0+
- J6 pad 16: A1+ -> A1-
- J6 pad 17: A1- -> A1+
- J6 pad 18: B1- -> B1+
- J6 pad 19: B1+ -> B1-
Routing:
- net B0+: track 5.09 -> 12.0 mm
- net B1-: track 5.55 -> 11.7 mm
- net A1-: track 3.28 -> 6.17 mm
- net A0+: track 3.35 -> 6.17 mm
- net A0-: track 3.57 -> 5.89 mm
- net A1+: track 3.63 -> 5.82 mm
- net B0-: track 9.42 -> 7.51 mm
- net GND: track 115.4 -> 117.1 mm, vias 13 -> 12
- net B1+: track 9.21 -> 7.96 mm
- net Net-(D1-Pad1): track 0.87 -> 2.05 mm
- net Net-(D2-Pad1): track 8.82 -> 8.17 mm
Other:
- outline, holes or cut-outs redrawn

Commit message: finished P4
Connections:
- J3 pad 12: B0-_top -> A0+_top
- J3 pad 14: A0+_top -> B0-_top
- J3 pad 16: A1+_top -> B1-_top
- J3 pad 18: B1-_top -> A1+_top
- J4 pad 50: A1+_top -> B1-_top
- J4 pad 60: B1-_top -> A1+_top
- J4 pad 64: B0-_top -> A0+_top
- J4 pad 68: A0+_top -> B0-_top
- J6 pad 12: B0+ -> A0+
- J6 pad 13: B0- -> B0+
- J6 pad 14: A0- -> B0-
- J6 pad 15: A0+ -> A0-
- J6 pad 16: A1- -> B1-
- J6 pad 17: A1+ -> A1-
- J6 pad 18: B1+ -> A1+
- J6 pad 19: B1- -> B1+
- U3 pad 1: A0+ -> A0-
- U3 pad 2: A0- -> B0-
- U3 pad 3: B0+ -> A0+
- U3 pad 4: B0- -> B0+
- U6 pad 1: A1+ -> A1-
- U6 pad 2: A1- -> B1-
- U6 pad 3: B1+ -> A1+
- U6 pad 4: B1- -> B1+
Routing:
- net A0+: track 6.17 -> 12.0 mm
- net B1-: track 11.7 -> 6.17 mm
- net B0+: track 12.0 -> 7.51 mm
- net B1+: track 7.96 -> 11.7 mm
- net B0-_top: track 6.65 -> 4.29 mm
- net A0+_top: track 4.29 -> 6.65 mm
- net B1-_top: track 18.0 -> 15.8 mm
- net A1+_top: track 15.8 -> 18.0 mm
- net A1+: track 5.82 -> 7.96 mm
- net B0-: track 7.51 -> 5.89 mm
