File: P4/PCB/MicroMod_tinycar/MicroMod_tinycar.sch (KiCad schematic (older format))
At the start: 13 parts

Commit message: p4 version1 pcb
Parts:
- removed C?: C_Small, symbol MicroMod_tinycar_symbol_library:C_Small
- removed D?: LED, symbol MicroMod_tinycar_symbol_library:LED
- removed J?: USB_B_Micro, symbol MicroMod_tinycar_symbol_library:USB_B_Micro
- removed L?: L_Small, symbol MicroMod_tinycar_symbol_library:L_Small
- removed Q?: DMG3415U, Package_DirectFET:DirectFET_MX, symbol MicroMod_tinycar_symbol_library:DMG3415U
- removed R?: R_Small, symbol MicroMod_tinycar_symbol_library:R_Small
- removed SW?: SW_Push, symbol MicroMod_tinycar_symbol_library:SW_Push
- removed U?: Boost_Converter_TPS61023, symbol MicroMod_tinycar_symbol_library:Boost_Converter_TPS61023
- removed U?: MCP73833-CNI_UN, SOP50P490X110-10N, symbol MicroMod_tinycar_symbol_library:MCP73833-CNI_UN
- added C1, C4: 4.7μ, MicroMod_tinycar_footprint_library:C_0805_2012Metric, symbol MicroMod_tinycar-rescue:C_Small-MicroMod_tinycar_symbol_library
- added C2, C3: 1μ, MicroMod_tinycar_footprint_library:C_0805_2012Metric, symbol MicroMod_tinycar-rescue:C_Small-MicroMod_tinycar_symbol_library
- added D1: R_LED, MicroMod_tinycar_footprint_library:LED_0805_2012Metric, symbol MicroMod_tinycar-rescue:LED-MicroMod_tinycar_symbol_library
- added D2: D_Schottky_Small, MicroMod_tinycar_footprint_library:D_0805_2012Metric, symbol MicroMod_tinycar-rescue:D_Schottky_Small
- added J1: USB_B_Micro, MicroMod_tinycar_footprint_library:USB_Micro-B_Molex_47346-0001, symbol MicroMod_tinycar-rescue:USB_B_Micro
- added J2: Conn_01x02, MicroMod_tinycar_footprint_library:JST_PH_S2B-PH-K_1x02_P2.00mm_Horizontal, symbol MicroMod_tinycar-rescue:Conn_01x02
- added J3, J6: Conn_02x15_Counter_Clockwise, MicroMod_tinycar_footprint_library:Bottom_adapter, symbol MicroMod_tinycar-rescue:Conn_02x15_Counter_Clockwise
- added J5: Conn_02x15_Counter_Clockwise, MicroMod_tinycar_footprint_library:Top_adapter, symbol MicroMod_tinycar-rescue:Conn_02x15_Counter_Clockwise
- added Q1: DMG2305UX-MicroMod_tinycar_symbol_library, MicroMod_tinycar_footprint_library:DMG2305UX_SOT-23, symbol MicroMod_tinycar-rescue:DMG2305UX-MicroMod_tinycar_symbol_library
- added R1, R6, R7: 10K, MicroMod_tinycar_footprint_library:R_0805_2012Metric, symbol MicroMod_tinycar-rescue:R_Small-MicroMod_tinycar_symbol_library
- added R2, R4: 5K, MicroMod_tinycar_footprint_library:R_0805_2012Metric, symbol MicroMod_tinycar-rescue:R_Small-MicroMod_tinycar_symbol_library
- added R3: 470, MicroMod_tinycar_footprint_library:R_0805_2012Metric, symbol MicroMod_tinycar-rescue:R_Small-MicroMod_tinycar_symbol_library
- added R5, R8: 100, MicroMod_tinycar_footprint_library:R_0805_2012Metric, symbol MicroMod_tinycar-rescue:R_Small-MicroMod_tinycar_symbol_library
- added U1: MCP73830LT-0AAI_MYY, MicroMod_tinycar_footprint_library:MCP73830LT-0AAI&slash_MYY, symbol MicroMod_tinycar-rescue:MCP73830LT-0AAI_MYY
- added U2: AP7333-SOT23R, MicroMod_tinycar_footprint_library:AP7333_SOT-23, symbol MicroMod_tinycar-rescue:AP7333-SOT23R
- added U3, U6: Stepper, MicroMod_tinycar_footprint_library:Mini_Stepper, symbol MicroMod_tinycar-rescue:Stepper
- added U4, U5: QRE1113GR, MicroMod_tinycar_footprint_library:QRE1113GR, symbol MicroMod_tinycar-rescue:QRE1113GR
- H1: renamed from H?; footprint (none) -> MicroMod_tinycar_footprint_library:STAND-OFF-REFLOW-M2.5; symbol MicroMod_tinycar_symbol_library:STAND-OFF-REFLOW2.5MM_TALL -> MicroMod_tinycar-rescue:STAND-OFF-REFLOW2.5MM_TALL-MicroMod_tinycar_symbol_library
- J4: renamed from J?; footprint (none) -> MicroMod_tinycar_footprint_library:M.2-CONNECTOR-E; symbol MicroMod_tinycar_symbol_library:MICROMOD-2222 -> MicroMod_tinycar-rescue:MICROMOD-2222-MicroMod_tinycar_symbol_library
- SW1: renamed from SW?; footprint (none) -> MicroMod_tinycar_footprint_library:SW_PCM12SMTR; symbol MicroMod_tinycar_symbol_library:SW_SPDT -> MicroMod_tinycar-rescue:SW_SPDT-MicroMod_tinycar_symbol_library
- SW2: renamed from SW?; footprint (none) -> MicroMod_tinycar_footprint_library:SW_TL1015AF160QG; symbol MicroMod_tinycar_symbol_library:SW_Push -> MicroMod_tinycar-rescue:SW_Push-MicroMod_tinycar_symbol_library
Connections:
- net labels added: 3V3_bot, A0+, A0+_top, A0-, A0-_top, A1+, A1+_top, A1-, A1-_top, B0+, B0+_top, B0-, B0-_top, B1+, B1+_top, B1-, B1-_top, CS, GND_bot, I2C_INT, Light0_bot, Light0_top, Light1_bot, Light1_top, PWM0, PWM1, RX1, SCK, SCL, SDA, SIPO, SOPI, SWDCK, SWDIO, TX1, USBHOST_D+, USBHOST_D-, VBATT_3
- wire segments 12 -> 191
- no-connect marks 1 -> 55
Other:
- note added: "Board to Board Connection"
- note added: "Lower Board"
- note added: "MicroMod Connection"
- note added: "Power Regulation"
- note added: "To Bottom Board"
- note added: "To Top Board(s)"
- note added: "USB Interface"

Commit message: done with P4
Parts:
- added U7: caster, MicroMod_tinycar_footprint_library:tiny_caster, symbol MicroMod_tinycar-rescue:caster
- added U8: MouseBite, MicroMod_tinycar_footprint_library:mouse-bite-2.54mm-slot, symbol MicroMod_tinycar-rescue:MouseBite
Connections:
- net A0+: now also J6.15 (Pin_15); no longer J6.14 (Pin_14)
- net A0-: now also J6.14 (Pin_14); no longer J6.15 (Pin_15)
- net A1+: now also J6.17 (Pin_17); no longer J6.16 (Pin_16)
- net A1-: now also J6.16 (Pin_16); no longer J6.17 (Pin_17)
- net B0+: now also J6.12 (Pin_12); no longer J6.13 (Pin_13)
- net B0-: now also J6.13 (Pin_13); no longer J6.12 (Pin_12)
- net B1+: now also J6.18 (Pin_18); no longer J6.19 (Pin_19)
- net B1-: now also J6.19 (Pin_19); no longer J6.18 (Pin_18)
- net PWM1: now also J5.21 (Pin_21)
- no-connect marks 55 -> 63
Other:
- note added: "MicroMod TinyCar\n"
- note added: "Panelization"
- moved on the sheet: J6, R5, R6, R7, R8, U3, U4, U5, U6

Commit message: finished P4
Parts:
- U3, U6: symbol MicroMod_tinycar-rescue:Stepper -> MicroMod_tinycar-rescue:Stepper-MicroMod_tinycar-rescue
Connections:
- net A0+: now also J6.12 (Pin_12), U3.3 (A+); no longer J6.15 (Pin_15), U3.1 (A+)
- net A0+_top: now also J3.12 (Pin_12), J4.64 (SPI_SDI1/SDIO_DATA0); no longer J3.14 (Pin_14), J4.68 (SDIO_DATA2)
- net A0-: now also J6.15 (Pin_15), U3.1 (A-); no longer J6.14 (Pin_14), U3.2 (A-)
- net A1+: now also J6.18 (Pin_18), U6.3 (A+); no longer J6.17 (Pin_17), U6.1 (A+)
- net A1+_top: now also J3.18 (Pin_18), J4.60 (SPI_SCK1/SDIO_CLK); no longer J3.16 (Pin_16), J4.50 (AUD_BCLK)
- net A1-: now also J6.17 (Pin_17), U6.1 (A-); no longer J6.16 (Pin_16), U6.2 (A-)
- net B0+: now also J6.13 (Pin_13), U3.4 (B+); no longer J6.12 (Pin_12), U3.3 (B+)
- net B0-: now also J6.14 (Pin_14), U3.2 (B-); no longer J6.13 (Pin_13), U3.4 (B-)
- net B0-_top: now also J3.14 (Pin_14), J4.68 (SDIO_DATA2); no longer J3.12 (Pin_12), J4.64 (SPI_SDI1/SDIO_DATA0)
- net B1+: now also J6.19 (Pin_19), U6.4 (B+); no longer J6.18 (Pin_18), U6.3 (B+)
- net B1-: now also J6.16 (Pin_16), U6.2 (B-); no longer J6.19 (Pin_19), U6.4 (B-)
- net B1-_top: now also J3.16 (Pin_16), J4.50 (AUD_BCLK); no longer J3.18 (Pin_18), J4.60 (SPI_SCK1/SDIO_CLK)
Changed lines of the file:
@@
 NoConn ~ 2500 7900
 $Comp
-L MicroMod_tinycar-rescue:Stepper U6
+L MicroMod_tinycar-rescue:Stepper-MicroMod_tinycar-rescue U6
 U 1 1 606EC968
 P 14800 3250
@@
 $EndComp
 $Comp
-L MicroMod_tinycar-rescue:Stepper U3
+L MicroMod_tinycar-rescue:Stepper-MicroMod_tinycar-rescue U3
 U 1 1 606ECEED
 P 13200 3150
@@
 	3700 8100 3750 8100
 Text GLabel 9750 5750 2    50   Input ~ 0
+B0-_top
+Text GLabel 9750 5550 2    50   Input ~ 0
 A0+_top
-Text GLabel 9750 5550 2    50   Input ~ 0
-B0-_top
 Text GLabel 9750 5650 2    50   Input ~ 0
 B0+_top
@@
 Wire Wire Line
 	9750 5850 9550 5850
-Text GLabel 9750 5350 2    50   Input ~ 0
+Text GLabel 7550 7750 0    50   Input ~ 0
 B1-_top
 Text GLabel 9750 5450 2    50   Input ~ 0
@@
 Text GLabel 7550 7650 0    50   Input ~ 0
 A1-_top
-Text GLabel 7550 7750 0    50   Input ~ 0
+Text GLabel 9750 5350 2    50   Input ~ 0
 A1+_top
 Wire Wire Line
@@
 NoConn ~ 9600 2450
 NoConn ~ 9600 2350
-Text GLabel 13600 2650 0    50   Input ~ 0
+Text GLabel 13600 2350 0    50   Input ~ 0
 A0+
-Text GLabel 13600 2550 0    50   Input ~ 0
-A0-
-Text GLabel 13600 2450 0    50   Input ~ 0
-B0-
-Text GLabel 13600 2350 0    50   Input ~ 0
-B0+
-Text GLabel 13550 3050 2    50   Input ~ 0
-A0+
-Text GLabel 13550 3150 2    50   Input ~ 0
-A0-
-Text GLabel 13550 3350 2    50   Input ~ 0
-B0-
-Text GLabel 13550 3250 2    50   Input ~ 0
-B0+
 Wire Wire Line
 	13600 2350 13750 2350
@@
 Wire Wire Line
 	13400 3150 13550 3150
-Text GLabel 14400 2550 2    50   Input ~ 0
-A1+
 Text GLabel 14400 2650 2    50   Input ~ 0
-A1-
+B1-
 Text GLabel 14400 2350 2    50   Input ~ 0
-B1-
+B1+
 Text GLabel 14400 2450 2    50   Input ~ 0
-B1+
-Text GLabel 14450 3350 0    50   Input ~ 0
 A1+
 Text GLabel 14450 3050 0    50   Input ~ 0
-B1-
+B1+
 Text GLabel 14450 3150 0    50   Input ~ 0
-B1+
-Text GLabel 14450 3250 0    50   Input ~ 0
-A1-
+A1+
 Wire Wire Line
 	14450 3050 14600 3050
@@
 Text GLabel 7700 2500 2    50   Input ~ 0
 B1+_top
+Text GLabel 7700 2800 2    50   Input ~ 0
+B1-_top
 Text GLabel 7700 2600 2    50   Input ~ 0
-B1-_top
-Text GLabel 7700 2800 2    50   Input ~ 0
 A1+_top
 Text GLabel 7700 2700 2    50   Input ~ 0
@@
 Text GLabel 6900 2600 0    50   Input ~ 0
 B0+_top
-Text GLabel 6900 2500 0    50   Input ~ 0
-B0-_top
-Text GLabel 6900 2700 0    50   Input ~ 0
-A0+_top
 Wire Wire Line
 	7550 2400 7700 2400
@@
 Text Notes 12750 10400 0    197  ~ 0
 MicroMod TinyCar\n
+Text GLabel 13550 3350 2    50   Input ~ 0
+B0+
+Text GLabel 13550 3250 2    50   Input ~ 0
+A0+
+Text GLabel 13550 3050 2    50   Input ~ 0
+A0-
+Text GLabel 13600 2650 0    50   Input ~ 0
+A0-
+Text GLabel 13550 3150 2    50   Input ~ 0
+B0-
+Text GLabel 14450 3250 0    50   Input ~ 0
+B1-
+Text GLabel 14400 2550 2    50   Input ~ 0
+A1-
+Text GLabel 14450 3350 0    50   Input ~ 0
+A1-
+Text GLabel 13600 2550 0    50   Input ~ 0
+B0-
+Text GLabel 13600 2450 0    50   Input ~ 0
+B0+
+Text GLabel 6900 2700 0    50   Input ~ 0
+B0-_top
+Text GLabel 6900 2500 0    50   Input ~ 0
+A0+_top
+Text GLabel 8150 2800 2    50   Input ~ 0
+B1-
+Text GLabel 8150 2500 2    50   Input ~ 0
+B1+
+Text GLabel 8150 2600 2    50   Input ~ 0
+A1+
+Text GLabel 8150 2700 2    50   Input ~ 0
+A1-
 $EndSCHEMATC
